File: KsbSchematics/KsbSchematics/KsbLightSensorSchematic.sch (EAGLE design)
At the start: 31 parts, among them IC1 7805L, IC2 LM311N, U1 ATTINY84

Commit message: schematics change
Connections:
- net +12V: now also R7.2
Changed lines of the file:
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@@
 <pinref part="C3" gate="G$1" pin="+"/>
 <wire x1="43.18" y1="124.46" x2="43.18" y2="165.1" width="0.1524" layer="91"/>
-<wire x1="43.18" y1="165.1" x2="93.98" y2="165.1" width="0.1524" layer="91"/>
+<wire x1="43.18" y1="165.1" x2="88.9" y2="165.1" width="0.1524" layer="91"/>
 <pinref part="R4" gate="G$1" pin="2"/>
 <pinref part="R8" gate="G$1" pin="2"/>
+<wire x1="88.9" y1="165.1" x2="93.98" y2="165.1" width="0.1524" layer="91"/>
 <wire x1="93.98" y1="165.1" x2="93.98" y2="157.48" width="0.1524" layer="91"/>
+<pinref part="R7" gate="G$1" pin="2"/>
+<wire x1="88.9" y1="165.1" x2="88.9" y2="157.48" width="0.1524" layer="91"/>
 </segment>
 <segment>
@@
 <pinref part="R10" gate="G$1" pin="1"/>
 <label x="-91.44" y="83.82" size="2.54" layer="95"/>
-<label x="-50.8" y="78.74" size="1.778" layer="95"/>
-</segment>
-</net>
+</segment>
+</net>

Commit message: reg save
Connections:
- new net N$19: SG1.1
Changed lines of the file:
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@@
 <net name="N$10" class="0">
 <segment>
-<wire x1="35.56" y1="71.12" x2="27.94" y2="71.12" width="0.1524" layer="91"/>
-<wire x1="27.94" y1="71.12" x2="27.94" y2="40.64" width="0.1524" layer="91"/>
+<wire x1="35.56" y1="68.58" x2="27.94" y2="68.58" width="0.1524" layer="91"/>
+<wire x1="27.94" y1="68.58" x2="27.94" y2="40.64" width="0.1524" layer="91"/>
 <wire x1="27.94" y1="40.64" x2="106.68" y2="40.64" width="0.1524" layer="91"/>
 <pinref part="R6" gate="G$1" pin="1"/>
@@
 <net name="N$11" class="0">
 <segment>
-<wire x1="35.56" y1="68.58" x2="30.48" y2="68.58" width="0.1524" layer="91"/>
-<wire x1="30.48" y1="68.58" x2="30.48" y2="50.8" width="0.1524" layer="91"/>
+<wire x1="35.56" y1="66.04" x2="30.48" y2="66.04" width="0.1524" layer="91"/>
+<wire x1="30.48" y1="66.04" x2="30.48" y2="50.8" width="0.1524" layer="91"/>
 <wire x1="30.48" y1="50.8" x2="106.68" y2="50.8" width="0.1524" layer="91"/>
 <pinref part="R5" gate="G$1" pin="1"/>
@@
 <wire x1="10.16" y1="10.16" x2="10.16" y2="5.08" width="0.1524" layer="91"/>
 <wire x1="10.16" y1="5.08" x2="25.4" y2="5.08" width="0.1524" layer="91"/>
-<wire x1="25.4" y1="5.08" x2="25.4" y2="35.56" width="0.1524" layer="91"/>
 <wire x1="10.16" y1="10.16" x2="10.16" y2="7.62" width="0.1524" layer="91"/>
 <junction x="10.16" y="10.16"/>
 <pinref part="OK1" gate="A" pin="COL"/>
 <pinref part="R14" gate="G$1" pin="1"/>
+<wire x1="25.4" y1="5.08" x2="25.4" y2="71.12" width="0.1524" layer="91"/>
+<wire x1="25.4" y1="71.12" x2="35.56" y2="71.12" width="0.1524" layer="91"/>
 </segment>
 </net>
@@
 </segment>
 </net>
+<net name="N$19" class="0">
+<segment>
+<pinref part="SG1" gate="G$1" pin="1"/>
+<wire x1="104.14" y1="83.82" x2="88.9" y2="83.82" width="0.1524" layer="91"/>
+<wire x1="88.9" y1="83.82" x2="88.9" y2="53.34" width="0.1524" layer="91"/>
+<wire x1="88.9" y1="53.34" x2="33.02" y2="53.34" width="0.1524" layer="91"/>
+<wire x1="33.02" y1="53.34" x2="33.02" y2="63.5" width="0.1524" layer="91"/>
+<wire x1="33.02" y1="63.5" x2="35.56" y2="63.5" width="0.1524" layer="91"/>
+</segment>
+</net>

Commit message: minor changes
Parts:
- added R16: (no value), resistor:R-EU_0613/5V
Connections:
- net +12V: now also R16.2
- net N$4: now also R16.1
Changed lines of the file:
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@@
 <part name="SUPPLY21" library="supply2" deviceset="GND" device=""/>
 <part name="R15" library="resistor" deviceset="R-EU_" device="0613/5V" value="2k"/>
+<part name="R16" library="resistor" deviceset="R-EU_" device="0613/5V"/>
+<part name="SUPPLY22" library="supply2" deviceset="+12V" device="" value="+5V"/>
 </parts>
 <sheets>
 <sheet>
 <plain>
-<rectangle x1="-40.64" y1="-12.7" x2="-38.1" y2="152.4" layer="91"/>
+<rectangle x1="-38.1" y1="-5.08" x2="-35.56" y2="160.02" layer="91"/>
 </plain>
 <instances>
@@
 <instance part="SUPPLY12" gate="GND" x="7.62" y="78.74"/>
 <instance part="SUPPLY13" gate="GND" x="7.62" y="40.64"/>
-<instance part="SUPPLY14" gate="GND" x="15.24" y="-55.88"/>
+<instance part="SUPPLY14" gate="GND" x="101.6" y="20.32"/>
 <instance part="SUPPLY15" gate="GND" x="-2.54" y="114.3"/>
 <instance part="LED1" gate="G$1" x="119.38" y="50.8" rot="R90"/>
@@
 <instance part="SUPPLY21" gate="GND" x="10.16" y="0"/>
 <instance part="R15" gate="G$1" x="-12.7" y="7.62"/>
+<instance part="R16" gate="G$1" x="147.32" y="139.7" rot="R90"/>
+<instance part="SUPPLY22" gate="+12V" x="147.32" y="147.32"/>
 </instances>
 <busses>
@@
 <net name="+12V" class="0">
 <segment>
+<pinref part="C3" gate="G$1" pin="+"/>
+<wire x1="12.7" y1="124.46" x2="35.56" y2="124.46" width="0.1524" layer="91"/>
+<junction x="12.7" y="124.46"/>
+<pinref part="SUPPLY2" gate="+12V" pin="+12V"/>
+<wire x1="10.16" y1="124.46" x2="12.7" y2="124.46" width="0.1524" layer="91"/>
+<junction x="10.16" y="124.46"/>
+<pinref part="C2" gate="G$1" pin="+"/>
 <wire x1="7.62" y1="124.46" x2="10.16" y2="124.46" width="0.1524" layer="91"/>
-<wire x1="10.16" y1="124.46" x2="12.7" y2="124.46" width="0.1524" layer="91"/>
-<wire x1="12.7" y1="124.46" x2="35.56" y2="124.46" width="0.1524" layer="91"/>
-<wire x1="35.56" y1="124.46" x2="43.18" y2="124.46" width="0.1524" layer="91"/>
-<junction x="12.7" y="124.46"/>
-<junction x="10.16" y="124.46"/>
-<junction x="35.56" y="124.46"/>
 <pinref part="IC1" gate="A1" pin="VO"/>
-<pinref part="SUPPLY2" gate="+12V" pin="+12V"/>
-<pinref part="C2" gate="G$1" pin="+"/>
-<pinref part="C3" gate="G$1" pin="+"/>
-<wire x1="43.18" y1="124.46" x2="43.18" y2="165.1" width="0.1524" layer="91"/>
-<wire x1="43.18" y1="165.1" x2="88.9" y2="165.1" width="0.1524" layer="91"/>
+<wire x1="35.56" y1="124.46" x2="35.56" y2="165.1" width="0.1524" layer="91"/>
 <pinref part="R4" gate="G$1" pin="2"/>
 <pinref part="R8" gate="G$1" pin="2"/>
-<wire x1="88.9" y1="165.1" x2="93.98" y2="165.1" width="0.1524" layer="91"/>
 <wire x1="93.98" y1="165.1" x2="93.98" y2="157.48" width="0.1524" layer="91"/>
+<wire x1="35.56" y1="165.1" x2="88.9" y2="165.1" width="0.1524" layer="91"/>
+<wire x1="93.98" y1="165.1" x2="88.9" y2="165.1" width="0.1524" layer="91"/>
 <pinref part="R7" gate="G$1" pin="2"/>
 <wire x1="88.9" y1="165.1" x2="88.9" y2="157.48" width="0.1524" layer="91"/>
@@
 <pinref part="SUPPLY20" gate="+12V" pin="+12V"/>
 </segment>
+<segment>
+<pinref part="R16" gate="G$1" pin="2"/>
+<pinref part="SUPPLY22" gate="+12V" pin="+12V"/>
+</segment>
 </net>
 <net name="GND" class="0">
@@
 </segment>
 <segment>
-<wire x1="15.24" y1="-53.34" x2="124.46" y2="-53.34" width="0.1524" layer="91"/>
-<wire x1="124.46" y1="-53.34" x2="124.46" y2="50.8" width="0.1524" layer="91"/>
+<wire x1="101.6" y1="22.86" x2="124.46" y2="22.86" width="0.1524" layer="91"/>
+<wire x1="124.46" y1="22.86" x2="124.46" y2="50.8" width="0.1524" layer="91"/>
 <pinref part="SUPPLY14" gate="GND" pin="GND"/>
 <pinref part="LED1" gate="G$1" pin="C"/>
@@
 <wire x1="154.94" y1="104.14" x2="30.48" y2="104.14" width="0.1524" layer="91"/>
 <wire x1="154.94" y1="134.62" x2="154.94" y2="104.14" width="0.1524" layer="91"/>
-<wire x1="139.7" y1="134.62" x2="154.94" y2="134.62" width="0.1524" layer="91"/>
+<wire x1="139.7" y1="134.62" x2="147.32" y2="134.62" width="0.1524" layer="91"/>
+<wire x1="147.32" y1="134.62" x2="154.94" y2="134.62" width="0.1524" layer="91"/>
 <wire x1="139.7" y1="134.62" x2="139.7" y2="121.92" width="0.1524" layer="91"/>
 <wire x1="139.7" y1="121.92" x2="137.16" y2="121.92" width="0.1524" layer="91"/>
@@
 <pinref part="IC2" gate="A" pin="OUT"/>
 <pinref part="R9" gate="G$1" pin="2"/>
-</segment>
-</net>
+<pinref part="R16" gate="G$1" pin="1"/>
+<junction x="147.32" y="134.62"/>
+</segment>
+</net>

Commit message: minor changes
Parts:
- removed R12, R13, R8, R9: (no value), resistor:R-EU_0613/5V
Connections:
- removed net N$14: R4.1, R8.1
- removed net N$17: R12.1, R2.E
- removed net N$18: R13.2, R2.A
- removed net N$7: IC2.-IN, R2.S, R9.1
- new net N$21: IC2.+IN, SENS-1.P$1
- net +12V: no longer R8.2
- net GND: now also R2.A; no longer R13.1
- net N$13: now also IC2.-IN, R2.S; no longer IC2.+IN, R12.2, R8.1, SENS-1.P$1
- net N$4: no longer R9.2
Other:
- moved on the sheet: R16
Changed lines of the file:
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@@
 <part name="R4" library="resistor" deviceset="R-EU_" device="0613/5V"/>
 <part name="R7" library="resistor" deviceset="R-EU_" device="0613/5V"/>
-<part name="R8" library="resistor" deviceset="R-EU_" device="0613/5V"/>
-<part name="R9" library="resistor" deviceset="R-EU_" device="0613/5V"/>
 <part name="R10" library="resistor" deviceset="R-EU_" device="0613/5V" value="2k"/>
 <part name="R11" library="resistor" deviceset="R-EU_" device="0613/5V" value="2k"/>
@@
 <part name="SUPPLY8" library="supply2" deviceset="GND" device=""/>
 <part name="SUPPLY11" library="supply2" deviceset="GND" device=""/>
-<part name="R12" library="resistor" deviceset="R-EU_" device="0613/5V"/>
-<part name="R13" library="resistor" deviceset="R-EU_" device="0613/5V"/>
 <part name="SUPPLY6" library="supply2" deviceset="GND" device=""/>
 <part name="SG1" library="buzzer" deviceset="EFB?" device="AA40D101"/>
@@
 <instance part="R4" gate="G$1" x="93.98" y="152.4" rot="R90"/>
 <instance part="R7" gate="G$1" x="88.9" y="152.4" rot="R90"/>
-<instance part="R8" gate="G$1" x="93.98" y="152.4" rot="R90"/>
-<instance part="R9" gate="G$1" x="132.08" y="121.92"/>
 <instance part="R10" gate="G$1" x="-15.24" y="86.36"/>
 <instance part="R11" gate="G$1" x="-15.24" y="48.26"/>
@@
 <instance part="SUPPLY8" gate="GND" x="-63.5" y="81.28"/>
 <instance part="SUPPLY11" gate="GND" x="-66.04" y="43.18"/>
-<instance part="R12" gate="G$1" x="116.84" y="142.24" rot="R90"/>
-<instance part="R13" gate="G$1" x="116.84" y="121.92" rot="R90"/>
 <instance part="SUPPLY6" gate="GND" x="116.84" y="114.3"/>
 <instance part="SG1" gate="G$1" x="106.68" y="86.36"/>
@@
 <instance part="SUPPLY21" gate="GND" x="10.16" y="0"/>
 <instance part="R15" gate="G$1" x="-12.7" y="7.62"/>
-<instance part="R16" gate="G$1" x="147.32" y="139.7" rot="R90"/>
-<instance part="SUPPLY22" gate="+12V" x="147.32" y="147.32"/>
+<instance part="R16" gate="G$1" x="154.94" y="139.7" rot="R90"/>
+<instance part="SUPPLY22" gate="+12V" x="154.94" y="147.32"/>
 </instances>
 <busses>
@@
 <wire x1="35.56" y1="124.46" x2="35.56" y2="165.1" width="0.1524" layer="91"/>
 <pinref part="R4" gate="G$1" pin="2"/>
-<pinref part="R8" gate="G$1" pin="2"/>
 <wire x1="93.98" y1="165.1" x2="93.98" y2="157.48" width="0.1524" layer="91"/>
 <wire x1="35.56" y1="165.1" x2="88.9" y2="165.1" width="0.1524" layer="91"/>
@@
 <pinref part="R7" gate="G$1" pin="2"/>
 <wire x1="88.9" y1="165.1" x2="88.9" y2="157.48" width="0.1524" layer="91"/>
+<wire x1="93.98" y1="165.1" x2="116.84" y2="165.1" width="0.1524" layer="91"/>
+<wire x1="116.84" y1="165.1" x2="116.84" y2="134.62" width="0.1524" layer="91"/>
 </segment>
 <segment>
@@
 </segment>
 <segment>
-<pinref part="R13" gate="G$1" pin="1"/>
-<pinref part="SUPPLY6" gate="GND" pin="GND"/>
-</segment>
-<segment>
 <pinref part="S3" gate="1" pin="S"/>
 <pinref part="SUPPLY18" gate="GND" pin="GND"/>
@@
 <pinref part="OK1" gate="A" pin="EMIT"/>
 <pinref part="SUPPLY21" gate="GND" pin="GND"/>
+</segment>
+<segment>
+<pinref part="R2" gate="1" pin="A"/>
+<pinref part="SUPPLY6" gate="GND" pin="GND"/>
+<wire x1="116.84" y1="127" x2="116.84" y2="116.84" width="0.1524" layer="91"/>
 </segment>
 </net>
@@
 </segment>
 </net>
-<net name="N$13" class="0">
-<segment>
-<wire x1="93.98" y1="147.32" x2="116.84" y2="147.32" width="0.1524" layer="91"/>
-<wire x1="116.84" y1="147.32" x2="114.3" y2="147.32" width="0.1524" layer="91"/>
-<wire x1="121.92" y1="147.32" x2="124.46" y2="147.32" width="0.1524" layer="91"/>
-<wire x1="124.46" y1="147.32" x2="124.46" y2="137.16" width="0.1524" layer="91"/>
-<wire x1="116.84" y1="147.32" x2="119.38" y2="147.32" width="0.1524" layer="91"/>
-<wire x1="121.92" y1="147.32" x2="119.38" y2="147.32" width="0.1524" layer="91"/>
-<junction x="116.84" y="147.32"/>
-<pinref part="SENS-1" gate="G$1" pin="P$1"/>
-<pinref part="R8" gate="G$1" pin="1"/>
-<pinref part="R12" gate="G$1" pin="2"/>
-<pinref part="IC2" gate="A" pin="+IN"/>
-</segment>
-</net>
-<net name="N$14" class="0">
-<segment>
-<pinref part="R4" gate="G$1" pin="1"/>
-<pinref part="R8" gate="G$1" pin="1"/>
-</segment>
-</net>
 <net name="N$4" class="0">
 <segment>
@@
 <wire x1="154.94" y1="104.14" x2="30.48" y2="104.14" width="0.1524" layer="91"/>
 <wire x1="154.94" y1="134.62" x2="154.94" y2="104.14" width="0.1524" layer="91"/>
-<wire x1="139.7" y1="134.62" x2="147.32" y2="134.62" width="0.1524" layer="91"/>
-<wire x1="147.32" y1="134.62" x2="154.94" y2="134.62" width="0.1524" layer="91"/>
-<wire x1="139.7" y1="134.62" x2="139.7" y2="121.92" width="0.1524" layer="91"/>
-<wire x1="139.7" y1="121.92" x2="137.16" y2="121.92" width="0.1524" layer="91"/>
+<wire x1="139.7" y1="134.62" x2="154.94" y2="134.62" width="0.1524" layer="91"/>
 <wire x1="30.48" y1="73.66" x2="35.56" y2="73.66" width="0.1524" layer="91"/>
 <wire x1="30.48" y1="81.28" x2="30.48" y2="73.66" width="0.1524" layer="91" curve="180"/>
 <pinref part="IC2" gate="A" pin="OUT"/>
-<pinref part="R9" gate="G$1" pin="2"/>
 <pinref part="R16" gate="G$1" pin="1"/>
-<junction x="147.32" y="134.62"/>
-</segment>
-</net>
-<net name="N$7" class="0">
-<segment>
-<wire x1="121.92" y1="132.08" x2="124.46" y2="132.08" width="0.1524" layer="91"/>
-<wire x1="127" y1="121.92" x2="121.92" y2="121.92" width="0.1524" layer="91"/>
-<wire x1="121.92" y1="121.92" x2="121.92" y2="132.08" width="0.1524" layer="91"/>
-<pinref part="R9" gate="G$1" pin="1"/>
-<pinref part="IC2" gate="A" pin="-IN"/>
-<pinref part="R2" gate="1" pin="S"/>
+<junction x="154.94" y="134.62"/>
 </segment>
 </net>
@@
 </segment>
 </net>
-<net name="N$17" class="0">
-<segment>
-<pinref part="R2" gate="1" pin="E"/>
-<pinref part="R12" gate="G$1" pin="1"/>
-</segment>
-</net>
-<net name="N$18" class="0">
-<segment>
-<pinref part="R2" gate="1" pin="A"/>
-<pinref part="R13" gate="G$1" pin="2"/>
-</segment>
-</net>
 <net name="N$5" class="0">
 <segment>
@@
 </segment>
 </net>
+<net name="N$21" class="0">
+<segment>
+<wire x1="114.3" y1="147.32" x2="119.38" y2="147.32" width="0.1524" layer="91" curve="-180"/>
+<wire x1="124.46" y1="147.32" x2="124.46" y2="137.16" width="0.1524" layer="91"/>
+<pinref part="IC2" gate="A" pin="+IN"/>
+<wire x1="119.38" y1="147.32" x2="124.46" y2="147.32" width="0.1524" layer="91"/>
+<pinref part="SENS-1" gate="G$1" pin="P$1"/>
+<wire x1="114.3" y1="147.32" x2="93.98" y2="147.32" width="0.1524" layer="91"/>
+</segment>
+</net>
+<net name="N$13" class="0">
+<segment>
+<pinref part="IC2" gate="A" pin="-IN"/>
+<wire x1="121.92" y1="132.08" x2="124.46" y2="132.08" width="0.1524" layer="91"/>
+<pinref part="R2" gate="1" pin="S"/>
+</segment>
+</net>

Commit message: minor changes
Parts:
- added DWIRE: (no value), con-lstb:MA03-2
Connections:
- net KSB-PULLED renamed D+
- new net N$7: DWIRE.5, U1.(!RESET!)PB3
- net +12V: now also DWIRE.2
- net GND: now also DWIRE.6
- net N$10: now also U1.(ADC3)PA3
- net N$15: now also U1.(ADC7)PA7
- net N$19: now also U1.(ADC1)PA1
- net N$4: now also U1.(RX/MISO/ADC5)PA5
- net N$6: now also U1.(TX/SDA/MOSI/ADC6)PA6
Changed lines of the file:
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@@
 <part name="R16" library="resistor" deviceset="R-EU_" device="0613/5V"/>
 <part name="SUPPLY22" library="supply2" deviceset="+12V" device="" value="+5V"/>
+<part name="SUPPLY23" library="supply2" deviceset="+12V" device="" value="+5V"/>
+<part name="SUPPLY24" library="supply2" deviceset="GND" device=""/>
+<part name="DWIRE" library="con-lstb" deviceset="MA03-2" device=""/>
 </parts>
 <sheets>
 <sheet>
 <plain>
-<rectangle x1="-38.1" y1="-5.08" x2="-35.56" y2="160.02" layer="91"/>
+<rectangle x1="-40.64" y1="-5.08" x2="-38.1" y2="160.02" layer="91"/>
 </plain>
 <instances>
@@
 <instance part="SENS-1" gate="G$1" x="91.44" y="137.16" rot="MR0"/>
 <instance part="SUPPLY1" gate="+12V" x="-66.04" y="127"/>
-<instance part="SUPPLY2" gate="+12V" x="12.7" y="127"/>
+<instance part="SUPPLY2" gate="+12V" x="17.78" y="127"/>
 <instance part="SUPPLY3" gate="+12V" x="-66.04" y="96.52"/>
 <instance part="S1" gate="1" x="-58.42" y="88.9" rot="MR270"/>
@@
 <instance part="R16" gate="G$1" x="154.94" y="139.7" rot="R90"/>
 <instance part="SUPPLY22" gate="+12V" x="154.94" y="147.32"/>
+<instance part="SUPPLY23" gate="+12V" x="167.64" y="88.9"/>
+<instance part="SUPPLY24" gate="GND" x="175.26" y="78.74"/>
+<instance part="DWIRE" gate="1" x="160.02" y="83.82" rot="R180"/>
 </instances>
 <busses>
@@
 <segment>
 <pinref part="C3" gate="G$1" pin="+"/>
-<wire x1="12.7" y1="124.46" x2="35.56" y2="124.46" width="0.1524" layer="91"/>
-<junction x="12.7" y="124.46"/>
+<wire x1="17.78" y1="124.46" x2="35.56" y2="124.46" width="0.1524" layer="91"/>
+<junction x="17.78" y="124.46"/>
 <pinref part="SUPPLY2" gate="+12V" pin="+12V"/>
-<wire x1="10.16" y1="124.46" x2="12.7" y2="124.46" width="0.1524" layer="91"/>
+<wire x1="10.16" y1="124.46" x2="17.78" y2="124.46" width="0.1524" layer="91"/>
 <junction x="10.16" y="124.46"/>
 <pinref part="C2" gate="G$1" pin="+"/>
 <wire x1="7.62" y1="124.46" x2="10.16" y2="124.46" width="0.1524" layer="91"/>
 <pinref part="IC1" gate="A1" pin="VO"/>
-<wire x1="35.56" y1="124.46" x2="35.56" y2="165.1" width="0.1524" layer="91"/>
+<wire x1="35.56" y1="124.46" x2="35.56" y2="157.48" width="0.1524" layer="91"/>
 <pinref part="R4" gate="G$1" pin="2"/>
-<wire x1="93.98" y1="165.1" x2="93.98" y2="157.48" width="0.1524" layer="91"/>
-<wire x1="35.56" y1="165.1" x2="88.9" y2="165.1" width="0.1524" layer="91"/>
-<wire x1="93.98" y1="165.1" x2="88.9" y2="165.1" width="0.1524" layer="91"/>
+<wire x1="35.56" y1="157.48" x2="88.9" y2="157.48" width="0.1524" layer="91"/>
+<wire x1="93.98" y1="157.48" x2="88.9" y2="157.48" width="0.1524" layer="91"/>
 <pinref part="R7" gate="G$1" pin="2"/>
-<wire x1="88.9" y1="165.1" x2="88.9" y2="157.48" width="0.1524" layer="91"/>
-<wire x1="93.98" y1="165.1" x2="116.84" y2="165.1" width="0.1524" layer="91"/>
-<wire x1="116.84" y1="165.1" x2="116.84" y2="134.62" width="0.1524" layer="91"/>
+<wire x1="93.98" y1="157.48" x2="116.84" y2="157.48" width="0.1524" layer="91"/>
+<wire x1="116.84" y1="157.48" x2="116.84" y2="134.62" width="0.1524" layer="91"/>
 </segment>
 <segment>
@@
 <pinref part="R16" gate="G$1" pin="2"/>
 <pinref part="SUPPLY22" gate="+12V" pin="+12V"/>
+</segment>
+<segment>
+<pinref part="SUPPLY23" gate="+12V" pin="+12V"/>
+<pinref part="DWIRE" gate="1" pin="2"/>
 </segment>
 </net>
@@
 <wire x1="116.84" y1="127" x2="116.84" y2="116.84" width="0.1524" layer="91"/>
 </segment>
+<segment>
+<pinref part="SUPPLY24" gate="GND" pin="GND"/>
+<wire x1="167.64" y1="81.28" x2="175.26" y2="81.28" width="0.1524" layer="91"/>
+<pinref part="DWIRE" gate="1" pin="6"/>
+</segment>
 </net>
 <net name="N$6" class="0">
@@
 <wire x1="7.62" y1="45.72" x2="22.86" y2="45.72" width="0.1524" layer="91"/>
 <wire x1="22.86" y1="45.72" x2="22.86" y2="76.2" width="0.1524" layer="91"/>
-<wire x1="22.86" y1="76.2" x2="38.1" y2="76.2" width="0.1524" layer="91"/>
+<wire x1="22.86" y1="76.2" x2="45.72" y2="76.2" width="0.1524" layer="91"/>
 <wire x1="7.62" y1="50.8" x2="7.62" y2="48.26" width="0.1524" layer="91"/>
 <junction x="7.62" y="50.8"/>
 <pinref part="OK4" gate="A" pin="COL"/>
 <pinref part="R3" gate="G$1" pin="1"/>
+<pinref part="U1" gate="U1" pin="(TX/SDA/MOSI/ADC6)PA6"/>
 </segment>
 </net>
@@
 <net name="N$10" class="0">
 <segment>
-<wire x1="35.56" y1="68.58" x2="27.94" y2="68.58" width="0.1524" layer="91"/>
 <wire x1="27.94" y1="68.58" x2="27.94" y2="40.64" width="0.1524" layer="91"/>
 <wire x1="27.94" y1="40.64" x2="106.68" y2="40.64" width="0.1524" layer="91"/>
 <pinref part="R6" gate="G$1" pin="1"/>
+<pinref part="U1" gate="U1" pin="(ADC3)PA3"/>
+<wire x1="27.94" y1="68.58" x2="45.72" y2="68.58" width="0.1524" layer="91"/>
 </segment>
 <segment>
@@
 <net name="N$11" class="0">
 <segment>
-<wire x1="35.56" y1="66.04" x2="30.48" y2="66.04" width="0.1524" layer="91"/>
 <wire x1="30.48" y1="66.04" x2="30.48" y2="50.8" width="0.1524" layer="91"/>
 <wire x1="30.48" y1="50.8" x2="106.68" y2="50.8" width="0.1524" layer="91"/>
 <pinref part="R5" gate="G$1" pin="1"/>
+<wire x1="30.48" y1="66.04" x2="48.26" y2="66.04" width="0.1524" layer="91"/>
 </segment>
 </net>
@@
 <wire x1="154.94" y1="134.62" x2="154.94" y2="104.14" width="0.1524" layer="91"/>
 <wire x1="139.7" y1="134.62" x2="154.94" y2="134.62" width="0.1524" layer="91"/>
-<wire x1="30.48" y1="73.66" x2="35.56" y2="73.66" width="0.1524" layer="91"/>
 <wire x1="30.48" y1="81.28" x2="30.48" y2="73.66" width="0.1524" layer="91" curve="180"/>
 <pinref part="IC2" gate="A" pin="OUT"/>
 <pinref part="R16" gate="G$1" pin="1"/>
 <junction x="154.94" y="134.62"/>
+<pinref part="U1" gate="U1" pin="(RX/MISO/ADC5)PA5"/>
+<wire x1="30.48" y1="73.66" x2="45.72" y2="73.66" width="0.1524" layer="91"/>
 </segment>
 </net>
@@
 <segment>
 <wire x1="7.62" y1="88.9" x2="7.62" y2="83.82" width="0.1524" layer="91"/>
-<wire x1="35.56" y1="78.74" x2="22.86" y2="78.74" width="0.1524" layer="91"/>
+<wire x1="45.72" y1="78.74" x2="22.86" y2="78.74" width="0.1524" layer="91"/>
 <wire x1="22.86" y1="78.74" x2="22.86" y2="83.82" width="0.1524" layer="91"/>
 <wire x1="22.86" y1="83.82" x2="7.62" y2="83.82" width="0.1524" layer="91"/>
@@
 <pinref part="OK3" gate="A" pin="COL"/>
 <pinref part="R1" gate="G$1" pin="1"/>
+<pinref part="U1" gate="U1" pin="(ADC7)PA7"/>
 </segment>
 </net>
@@
 </segment>
 </net>
-<net name="KSB-PULLED" class="0">
+<net name="D+" class="0">
 <segment>
 <wire x1="-53.34" y1="86.36" x2="-20.32" y2="86.36" width="0.1524" layer="91"/>
 <pinref part="S1" gate="1" pin="P"/>
 <pinref part="R10" gate="G$1" pin="1"/>
-<label x="-91.44" y="83.82" size="2.54" layer="95"/>
+<label x="-78.74" y="83.82" size="2.54" layer="95"/>
 </segment>
 </net>
@@
 <pinref part="R14" gate="G$1" pin="1"/>
 <wire x1="25.4" y1="5.08" x2="25.4" y2="71.12" width="0.1524" layer="91"/>
-<wire x1="25.4" y1="71.12" x2="35.56" y2="71.12" width="0.1524" layer="91"/>
+<wire x1="25.4" y1="71.12" x2="33.02" y2="71.12" width="0.1524" layer="91"/>
+<wire x1="33.02" y1="71.12" x2="35.56" y2="71.12" width="0.1524" layer="91"/>
+<wire x1="35.56" y1="71.12" x2="48.26" y2="71.12" width="0.1524" layer="91"/>
 </segment>
 </net>
@@
 <wire x1="88.9" y1="53.34" x2="33.02" y2="53.34" width="0.1524" layer="91"/>
 <wire x1="33.02" y1="53.34" x2="33.02" y2="63.5" width="0.1524" layer="91"/>
-<wire x1="33.02" y1="63.5" x2="35.56" y2="63.5" width="0.1524" layer="91"/>
+<pinref part="U1" gate="U1" pin="(ADC1)PA1"/>
+<wire x1="33.02" y1="63.5" x2="45.72" y2="63.5" width="0.1524" layer="91"/>
 </segment>
 </net>
@@
 </segment>
 </net>
+<net name="N$7" class="0">
+<segment>
+<pinref part="U1" gate="U1" pin="(!RESET!)PB3"/>
+<wire x1="45.72" y1="91.44" x2="40.64" y2="91.44" width="0.1524" layer="91"/>
+<wire x1="40.64" y1="91.44" x2="40.64" y2="99.06" width="0.1524" layer="91"/>
+<wire x1="40.64" y1="99.06" x2="142.24" y2="99.06" width="0.1524" layer="91"/>
+<wire x1="142.24" y1="99.06" x2="142.24" y2="81.28" width="0.1524" layer="91"/>
+<wire x1="142.24" y1="81.28" x2="152.4" y2="81.28" width="0.1524" layer="91"/>
+<pinref part="DWIRE" gate="1" pin="5"/>
+<wire x1="152.4" y1="81.28" x2="154.94" y2="81.28" width="0.1524" layer="91"/>
+<junction x="152.4" y="81.28"/>
+</segment>
+</net>
