File: KsbSchematics/KsbSchematics/KsbLightSensorSchematic.sch (EAGLE design)
At the start: 29 parts, among them IC1 7805L, IC2 LM311N, U1 ATTINY84

Commit message: minor changes
Connections:
- net GND: now also LED2.C, SG1.2
Other:
- moved on the sheet: DWIRE, LED1, LED2, R5, R6, SG1
Changed lines of the file:
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@@
 <instance part="SUPPLY12" gate="GND" x="7.62" y="78.74"/>
 <instance part="SUPPLY13" gate="GND" x="7.62" y="40.64"/>
-<instance part="SUPPLY14" gate="GND" x="101.6" y="20.32"/>
+<instance part="SUPPLY14" gate="GND" x="124.46" y="7.62"/>
 <instance part="SUPPLY15" gate="GND" x="-2.54" y="114.3"/>
-<instance part="LED1" gate="G$1" x="119.38" y="50.8" rot="R90"/>
-<instance part="LED2" gate="G$1" x="119.38" y="40.64" rot="R90"/>
-<instance part="R5" gate="G$1" x="111.76" y="50.8"/>
-<instance part="R6" gate="G$1" x="111.76" y="40.64"/>
-<instance part="SUPPLY17" gate="GND" x="111.76" y="81.28"/>
+<instance part="LED1" gate="G$1" x="142.24" y="27.94" rot="R90"/>
+<instance part="LED2" gate="G$1" x="142.24" y="17.78" rot="R90"/>
+<instance part="R5" gate="G$1" x="134.62" y="27.94"/>
+<instance part="R6" gate="G$1" x="134.62" y="17.78"/>
+<instance part="SUPPLY17" gate="GND" x="111.76" y="78.74"/>
 <instance part="R4" gate="G$1" x="93.98" y="152.4" rot="R90"/>
 <instance part="R7" gate="G$1" x="88.9" y="152.4" rot="R90"/>
@@
 <instance part="SUPPLY8" gate="GND" x="-63.5" y="81.28"/>
 <instance part="SUPPLY11" gate="GND" x="-66.04" y="43.18"/>
-<instance part="SUPPLY6" gate="GND" x="116.84" y="114.3"/>
-<instance part="SG1" gate="G$1" x="106.68" y="86.36"/>
+<instance part="SUPPLY6" gate="GND" x="116.84" y="124.46"/>
+<instance part="SG1" gate="G$1" x="106.68" y="83.82"/>
 <instance part="U1" gate="U1" x="63.5" y="76.2" rot="MR0"/>
 <instance part="SUPPLY16" gate="+12V" x="-68.58" y="17.78"/>
@@
 <instance part="R16" gate="G$1" x="154.94" y="139.7" rot="R90"/>
 <instance part="SUPPLY22" gate="+12V" x="154.94" y="147.32"/>
-<instance part="SUPPLY23" gate="+12V" x="167.64" y="88.9"/>
-<instance part="SUPPLY24" gate="GND" x="175.26" y="78.74"/>
-<instance part="DWIRE" gate="1" x="160.02" y="83.82" rot="R180"/>
+<instance part="SUPPLY23" gate="+12V" x="132.08" y="63.5"/>
+<instance part="SUPPLY24" gate="GND" x="139.7" y="53.34"/>
+<instance part="DWIRE" gate="1" x="124.46" y="58.42" rot="R180"/>
 </instances>
 <busses>
@@
 </segment>
 <segment>
-<wire x1="101.6" y1="22.86" x2="124.46" y2="22.86" width="0.1524" layer="91"/>
-<wire x1="124.46" y1="22.86" x2="124.46" y2="50.8" width="0.1524" layer="91"/>
-<pinref part="SUPPLY14" gate="GND" pin="GND"/>
-<pinref part="LED1" gate="G$1" pin="C"/>
-</segment>
-<segment>
 <wire x1="-2.54" y1="116.84" x2="10.16" y2="116.84" width="0.1524" layer="91"/>
 <wire x1="10.16" y1="116.84" x2="35.56" y2="116.84" width="0.1524" layer="91"/>
-<wire x1="35.56" y1="116.84" x2="43.18" y2="116.84" width="0.1524" layer="91"/>
-<wire x1="43.18" y1="116.84" x2="43.18" y2="109.22" width="0.1524" layer="91"/>
-<wire x1="43.18" y1="109.22" x2="88.9" y2="109.22" width="0.1524" layer="91"/>
-<wire x1="88.9" y1="109.22" x2="93.98" y2="109.22" width="0.1524" layer="91"/>
-<wire x1="88.9" y1="127" x2="88.9" y2="109.22" width="0.1524" layer="91"/>
-<wire x1="93.98" y1="127" x2="93.98" y2="109.22" width="0.1524" layer="91"/>
+<wire x1="35.56" y1="116.84" x2="88.9" y2="116.84" width="0.1524" layer="91"/>
+<wire x1="88.9" y1="116.84" x2="93.98" y2="116.84" width="0.1524" layer="91"/>
+<wire x1="88.9" y1="127" x2="88.9" y2="116.84" width="0.1524" layer="91"/>
+<wire x1="93.98" y1="127" x2="93.98" y2="116.84" width="0.1524" layer="91"/>
 <wire x1="93.98" y1="129.54" x2="93.98" y2="127" width="0.1524" layer="91"/>
 <wire x1="-2.54" y1="116.84" x2="-15.24" y2="116.84" width="0.1524" layer="91"/>
@@
 <pinref part="R2" gate="1" pin="A"/>
 <pinref part="SUPPLY6" gate="GND" pin="GND"/>
-<wire x1="116.84" y1="127" x2="116.84" y2="116.84" width="0.1524" layer="91"/>
 </segment>
 <segment>
 <pinref part="SUPPLY24" gate="GND" pin="GND"/>
-<wire x1="167.64" y1="81.28" x2="175.26" y2="81.28" width="0.1524" layer="91"/>
+<wire x1="132.08" y1="55.88" x2="139.7" y2="55.88" width="0.1524" layer="91"/>
 <pinref part="DWIRE" gate="1" pin="6"/>
+</segment>
+<segment>
+<pinref part="SG1" gate="G$1" pin="2"/>
+<pinref part="SUPPLY17" gate="GND" pin="GND"/>
+</segment>
+<segment>
+<wire x1="147.32" y1="10.16" x2="147.32" y2="17.78" width="0.1524" layer="91"/>
+<pinref part="LED1" gate="G$1" pin="C"/>
+<pinref part="LED2" gate="G$1" pin="C"/>
+<wire x1="147.32" y1="17.78" x2="147.32" y2="27.94" width="0.1524" layer="91"/>
+<junction x="147.32" y="17.78"/>
+<pinref part="SUPPLY14" gate="GND" pin="GND"/>
+<wire x1="124.46" y1="10.16" x2="147.32" y2="10.16" width="0.1524" layer="91"/>
 </segment>
 </net>
@@
 <net name="N$10" class="0">
 <segment>
-<wire x1="27.94" y1="68.58" x2="27.94" y2="40.64" width="0.1524" layer="91"/>
-<wire x1="27.94" y1="40.64" x2="106.68" y2="40.64" width="0.1524" layer="91"/>
+<wire x1="27.94" y1="68.58" x2="27.94" y2="17.78" width="0.1524" layer="91"/>
+<wire x1="27.94" y1="17.78" x2="129.54" y2="17.78" width="0.1524" layer="91"/>
 <pinref part="R6" gate="G$1" pin="1"/>
 <pinref part="U1" gate="U1" pin="(ADC3)PA3"/>
@@
 <net name="N$11" class="0">
 <segment>
-<wire x1="30.48" y1="66.04" x2="30.48" y2="50.8" width="0.1524" layer="91"/>
-<wire x1="30.48" y1="50.8" x2="106.68" y2="50.8" width="0.1524" layer="91"/>
+<wire x1="30.48" y1="66.04" x2="30.48" y2="27.94" width="0.1524" layer="91"/>
+<wire x1="30.48" y1="27.94" x2="129.54" y2="27.94" width="0.1524" layer="91"/>
 <pinref part="R5" gate="G$1" pin="1"/>
 <wire x1="30.48" y1="66.04" x2="48.26" y2="66.04" width="0.1524" layer="91"/>
@@
 <segment>
 <pinref part="SG1" gate="G$1" pin="1"/>
-<wire x1="104.14" y1="83.82" x2="88.9" y2="83.82" width="0.1524" layer="91"/>
-<wire x1="88.9" y1="83.82" x2="88.9" y2="53.34" width="0.1524" layer="91"/>
+<wire x1="104.14" y1="81.28" x2="88.9" y2="81.28" width="0.1524" layer="91"/>
+<wire x1="88.9" y1="81.28" x2="88.9" y2="53.34" width="0.1524" layer="91"/>
 <wire x1="88.9" y1="53.34" x2="33.02" y2="53.34" width="0.1524" layer="91"/>
 <wire x1="33.02" y1="53.34" x2="33.02" y2="63.5" width="0.1524" layer="91"/>
@@
 <pinref part="U1" gate="U1" pin="(!RESET!)PB3"/>
 <wire x1="45.72" y1="91.44" x2="40.64" y2="91.44" width="0.1524" layer="91"/>
-<wire x1="40.64" y1="91.44" x2="40.64" y2="99.06" width="0.1524" layer="91"/>
-<wire x1="40.64" y1="99.06" x2="142.24" y2="99.06" width="0.1524" layer="91"/>
-<wire x1="142.24" y1="99.06" x2="142.24" y2="81.28" width="0.1524" layer="91"/>
-<wire x1="142.24" y1="81.28" x2="152.4" y2="81.28" width="0.1524" layer="91"/>
+<wire x1="40.64" y1="91.44" x2="40.64" y2="96.52" width="0.1524" layer="91"/>
+<wire x1="40.64" y1="96.52" x2="137.16" y2="96.52" width="0.1524" layer="91"/>
+<wire x1="137.16" y1="96.52" x2="137.16" y2="71.12" width="0.1524" layer="91"/>
+<wire x1="137.16" y1="71.12" x2="109.22" y2="71.12" width="0.1524" layer="91"/>
 <pinref part="DWIRE" gate="1" pin="5"/>
-<wire x1="152.4" y1="81.28" x2="154.94" y2="81.28" width="0.1524" layer="91"/>
-<junction x="152.4" y="81.28"/>
-</segment>
-</net>
+<wire x1="116.84" y1="55.88" x2="119.38" y2="55.88" width="0.1524" layer="91"/>
+<junction x="116.84" y="55.88"/>
+<wire x1="109.22" y1="55.88" x2="116.84" y2="55.88" width="0.1524" layer="91"/>
+<wire x1="109.22" y1="71.12" x2="109.22" y2="55.88" width="0.1524" layer="91"/>
+</segment>
+</net>

Commit message: schematic changes
Connections:
- net N$11 renamed LED-BOARD
- net N$21 renamed CPU-BOARD
- new net ENTRY-BOARD: C2.+, C3.+, IC1.VO, R4.2, R7.2
- net +12V: no longer C2.+, C3.+, IC1.VO, R4.2, R7.2
Other:
- moved on the sheet: C3
Changed lines of the file:
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@@
 <plain>
 <rectangle x1="-40.64" y1="-5.08" x2="-38.1" y2="160.02" layer="91"/>
+<rectangle x1="-30.48" y1="-5.08" x2="27.94" y2="154.94" layer="207"/>
+<polygon width="0.1524" layer="207">
+<vertex x="104.14" y="116.84"/>
+<vertex x="104.14" y="162.56"/>
+<vertex x="170.18" y="162.56"/>
+<vertex x="162.56" y="162.56"/>
+<vertex x="162.56" y="45.72"/>
+<vertex x="40.64" y="45.72"/>
+<vertex x="38.1" y="45.72"/>
+<vertex x="38.1" y="109.22"/>
+<vertex x="104.14" y="109.22"/>
+<vertex x="104.14" y="111.76"/>
+</polygon>
+<rectangle x1="111.76" y1="-2.54" x2="162.56" y2="35.56" layer="207"/>
 </plain>
 <instances>
@@
 <instance part="C1" gate="G$1" x="-15.24" y="121.92"/>
 <instance part="C2" gate="G$1" x="10.16" y="121.92"/>
-<instance part="C3" gate="G$1" x="35.56" y="121.92"/>
+<instance part="C3" gate="G$1" x="22.86" y="121.92"/>
 <instance part="SUPPLY8" gate="GND" x="-63.5" y="81.28"/>
 <instance part="SUPPLY11" gate="GND" x="-66.04" y="43.18"/>
@@
 <net name="+12V" class="0">
 <segment>
-<pinref part="C3" gate="G$1" pin="+"/>
-<wire x1="17.78" y1="124.46" x2="35.56" y2="124.46" width="0.1524" layer="91"/>
-<junction x="17.78" y="124.46"/>
-<pinref part="SUPPLY2" gate="+12V" pin="+12V"/>
-<wire x1="10.16" y1="124.46" x2="17.78" y2="124.46" width="0.1524" layer="91"/>
-<junction x="10.16" y="124.46"/>
-<pinref part="C2" gate="G$1" pin="+"/>
-<wire x1="7.62" y1="124.46" x2="10.16" y2="124.46" width="0.1524" layer="91"/>
-<pinref part="IC1" gate="A1" pin="VO"/>
-<wire x1="35.56" y1="124.46" x2="35.56" y2="157.48" width="0.1524" layer="91"/>
-<pinref part="R4" gate="G$1" pin="2"/>
-<wire x1="35.56" y1="157.48" x2="88.9" y2="157.48" width="0.1524" layer="91"/>
-<wire x1="93.98" y1="157.48" x2="88.9" y2="157.48" width="0.1524" layer="91"/>
-<pinref part="R7" gate="G$1" pin="2"/>
-<wire x1="93.98" y1="157.48" x2="116.84" y2="157.48" width="0.1524" layer="91"/>
-<wire x1="116.84" y1="157.48" x2="116.84" y2="134.62" width="0.1524" layer="91"/>
-</segment>
-<segment>
 <wire x1="-66.04" y1="93.98" x2="-66.04" y2="88.9" width="0.1524" layer="91"/>
 <wire x1="-66.04" y1="88.9" x2="-63.5" y2="88.9" width="0.1524" layer="91"/>
@@
 <segment>
 <wire x1="-2.54" y1="116.84" x2="10.16" y2="116.84" width="0.1524" layer="91"/>
-<wire x1="10.16" y1="116.84" x2="35.56" y2="116.84" width="0.1524" layer="91"/>
-<wire x1="35.56" y1="116.84" x2="88.9" y2="116.84" width="0.1524" layer="91"/>
+<wire x1="10.16" y1="116.84" x2="22.86" y2="116.84" width="0.1524" layer="91"/>
+<wire x1="22.86" y1="116.84" x2="88.9" y2="116.84" width="0.1524" layer="91"/>
 <wire x1="88.9" y1="116.84" x2="93.98" y2="116.84" width="0.1524" layer="91"/>
 <wire x1="88.9" y1="127" x2="88.9" y2="116.84" width="0.1524" layer="91"/>
@@
 <junction x="-2.54" y="116.84"/>
 <junction x="10.16" y="116.84"/>
-<junction x="35.56" y="116.84"/>
+<junction x="22.86" y="116.84"/>
 <pinref part="IC1" gate="A1" pin="GND"/>
 <pinref part="SUPPLY15" gate="GND" pin="GND"/>
@@
 </segment>
 </net>
-<net name="N$11" class="0">
+<net name="LED-BOARD" class="0">
 <segment>
 <wire x1="30.48" y1="66.04" x2="30.48" y2="27.94" width="0.1524" layer="91"/>
@@
 <pinref part="R5" gate="G$1" pin="1"/>
 <wire x1="30.48" y1="66.04" x2="48.26" y2="66.04" width="0.1524" layer="91"/>
+<label x="129.54" y="38.1" size="3.048" layer="95"/>
 </segment>
 </net>
@@
 </segment>
 </net>
-<net name="N$21" class="0">
+<net name="CPU-BOARD" class="0">
 <segment>
 <wire x1="114.3" y1="147.32" x2="119.38" y2="147.32" width="0.1524" layer="91" curve="-180"/>
@@
 <pinref part="SENS-1" gate="G$1" pin="P$1"/>
 <wire x1="114.3" y1="147.32" x2="93.98" y2="147.32" width="0.1524" layer="91"/>
+<label x="111.76" y="165.1" size="3.048" layer="95"/>
 </segment>
 </net>
@@
 </segment>
 </net>
+<net name="ENTRY-BOARD" class="0">
+<segment>
+<pinref part="C3" gate="G$1" pin="+"/>
+<wire x1="17.78" y1="124.46" x2="22.86" y2="124.46" width="0.1524" layer="91"/>
+<junction x="17.78" y="124.46"/>
+<pinref part="SUPPLY2" gate="+12V" pin="+12V"/>
+<wire x1="10.16" y1="124.46" x2="17.78" y2="124.46" width="0.1524" layer="91"/>
+<junction x="10.16" y="124.46"/>
+<pinref part="C2" gate="G$1" pin="+"/>
+<wire x1="7.62" y1="124.46" x2="10.16" y2="124.46" width="0.1524" layer="91"/>
+<pinref part="IC1" gate="A1" pin="VO"/>
+<pinref part="R4" gate="G$1" pin="2"/>
+<wire x1="35.56" y1="157.48" x2="88.9" y2="157.48" width="0.1524" layer="91"/>
+<wire x1="93.98" y1="157.48" x2="88.9" y2="157.48" width="0.1524" layer="91"/>
+<pinref part="R7" gate="G$1" pin="2"/>
+<wire x1="93.98" y1="157.48" x2="116.84" y2="157.48" width="0.1524" layer="91"/>
+<wire x1="116.84" y1="157.48" x2="116.84" y2="134.62" width="0.1524" layer="91"/>
+<wire x1="35.56" y1="157.48" x2="35.56" y2="124.46" width="0.1524" layer="91"/>
+<wire x1="35.56" y1="124.46" x2="22.86" y2="124.46" width="0.1524" layer="91"/>
+<label x="7.62" y="157.48" size="3.302" layer="95" rot="MR0"/>
+</segment>
+</net>

Commit message: schematic changes
Changed lines of the file:
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@@
 <part name="SUPPLY24" library="supply2" deviceset="GND" device=""/>
 <part name="DWIRE" library="con-lstb" deviceset="MA03-2" device=""/>
+<part name="SUPPLY25" library="supply2" deviceset="GND" device=""/>
 </parts>
 <sheets>
@@
 <instance part="SUPPLY24" gate="GND" x="139.7" y="53.34"/>
 <instance part="DWIRE" gate="1" x="124.46" y="58.42" rot="R180"/>
+<instance part="SUPPLY25" gate="GND" x="-66.04" y="114.3"/>
 </instances>
 <busses>
@@
 <pinref part="C2" gate="G$1" pin="-"/>
 <pinref part="C3" gate="G$1" pin="-"/>
+<wire x1="-15.24" y1="116.84" x2="-66.04" y2="116.84" width="0.1524" layer="91"/>
+<pinref part="SUPPLY25" gate="GND" pin="GND"/>
 </segment>
 <segment>
@@
 <wire x1="-15.24" y1="124.46" x2="-12.7" y2="124.46" width="0.1524" layer="91"/>
 <junction x="-15.24" y="124.46"/>
-<label x="-83.82" y="116.84" size="2.54" layer="95" xref="yes"/>
+<label x="-106.68" y="114.3" size="2.54" layer="95" xref="yes"/>
 <pinref part="IC1" gate="A1" pin="VI"/>
 <pinref part="SUPPLY1" gate="+12V" pin="+12V"/>
