File: KsbSchematics/KsbSchematics/KsbLightSensorSchematic.sch (EAGLE design)
At the start: 29 parts, among them IC1 7805L, IC2 LM311N, U1 ATTINY84

Commit message: schematic changes
Connections:
- net N$15: now also U1.(TX/SDA/MOSI/ADC6)PA6; no longer U1.(ADC7)PA7
- net N$4: no longer U1.(RX/MISO/ADC5)PA5
- net N$6: now also U1.(RX/MISO/ADC5)PA5; no longer U1.(TX/SDA/MOSI/ADC6)PA6
Changed lines of the file:
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@@
 <rectangle x1="-30.48" y1="-5.08" x2="27.94" y2="154.94" layer="207"/>
 <polygon width="0.1524" layer="207">
-<vertex x="104.14" y="116.84"/>
+<vertex x="104.14" y="109.22"/>
 <vertex x="104.14" y="162.56"/>
 <vertex x="170.18" y="162.56"/>
 <vertex x="162.56" y="162.56"/>
 <vertex x="162.56" y="45.72"/>
-<vertex x="40.64" y="45.72"/>
-<vertex x="38.1" y="45.72"/>
-<vertex x="38.1" y="109.22"/>
-<vertex x="104.14" y="109.22"/>
-<vertex x="104.14" y="111.76"/>
+<vertex x="30.48" y="43.18"/>
+<vertex x="30.48" y="109.22"/>
 </polygon>
 <rectangle x1="111.76" y1="-2.54" x2="162.56" y2="35.56" layer="207"/>
@@
 <wire x1="7.62" y1="50.8" x2="7.62" y2="45.72" width="0.1524" layer="91"/>
 <wire x1="7.62" y1="45.72" x2="22.86" y2="45.72" width="0.1524" layer="91"/>
-<wire x1="22.86" y1="45.72" x2="22.86" y2="76.2" width="0.1524" layer="91"/>
-<wire x1="22.86" y1="76.2" x2="45.72" y2="76.2" width="0.1524" layer="91"/>
 <wire x1="7.62" y1="50.8" x2="7.62" y2="48.26" width="0.1524" layer="91"/>
 <junction x="7.62" y="50.8"/>
 <pinref part="OK4" gate="A" pin="COL"/>
 <pinref part="R3" gate="G$1" pin="1"/>
-<pinref part="U1" gate="U1" pin="(TX/SDA/MOSI/ADC6)PA6"/>
+<wire x1="22.86" y1="45.72" x2="22.86" y2="73.66" width="0.1524" layer="91"/>
+<pinref part="U1" gate="U1" pin="(RX/MISO/ADC5)PA5"/>
+<wire x1="45.72" y1="73.66" x2="38.1" y2="73.66" width="0.1524" layer="91"/>
+<wire x1="38.1" y1="73.66" x2="35.56" y2="73.66" width="0.1524" layer="91"/>
+<wire x1="22.86" y1="73.66" x2="35.56" y2="73.66" width="0.1524" layer="91"/>
 </segment>
 </net>
@@
 <net name="N$10" class="0">
 <segment>
-<wire x1="27.94" y1="68.58" x2="27.94" y2="17.78" width="0.1524" layer="91"/>
-<wire x1="27.94" y1="17.78" x2="129.54" y2="17.78" width="0.1524" layer="91"/>
+<wire x1="38.1" y1="68.58" x2="38.1" y2="17.78" width="0.1524" layer="91"/>
+<wire x1="38.1" y1="17.78" x2="129.54" y2="17.78" width="0.1524" layer="91"/>
 <pinref part="R6" gate="G$1" pin="1"/>
 <pinref part="U1" gate="U1" pin="(ADC3)PA3"/>
-<wire x1="27.94" y1="68.58" x2="45.72" y2="68.58" width="0.1524" layer="91"/>
-</segment>
-<segment>
-<wire x1="22.86" y1="76.2" x2="22.86" y2="45.72" width="0.1524" layer="91"/>
-</segment>
-<segment>
-<wire x1="22.86" y1="76.2" x2="22.86" y2="45.72" width="0.1524" layer="91"/>
+<wire x1="38.1" y1="68.58" x2="45.72" y2="68.58" width="0.1524" layer="91"/>
 </segment>
 </net>
 <net name="LED-BOARD" class="0">
 <segment>
-<wire x1="30.48" y1="66.04" x2="30.48" y2="27.94" width="0.1524" layer="91"/>
-<wire x1="30.48" y1="27.94" x2="129.54" y2="27.94" width="0.1524" layer="91"/>
+<wire x1="40.64" y1="66.04" x2="40.64" y2="27.94" width="0.1524" layer="91"/>
+<wire x1="40.64" y1="27.94" x2="129.54" y2="27.94" width="0.1524" layer="91"/>
 <pinref part="R5" gate="G$1" pin="1"/>
-<wire x1="30.48" y1="66.04" x2="48.26" y2="66.04" width="0.1524" layer="91"/>
+<wire x1="40.64" y1="66.04" x2="48.26" y2="66.04" width="0.1524" layer="91"/>
 <label x="129.54" y="38.1" size="3.048" layer="95"/>
 </segment>
@@
 <net name="N$4" class="0">
 <segment>
-<wire x1="30.48" y1="104.14" x2="30.48" y2="81.28" width="0.1524" layer="91"/>
-<wire x1="154.94" y1="104.14" x2="30.48" y2="104.14" width="0.1524" layer="91"/>
 <wire x1="154.94" y1="134.62" x2="154.94" y2="104.14" width="0.1524" layer="91"/>
 <wire x1="139.7" y1="134.62" x2="154.94" y2="134.62" width="0.1524" layer="91"/>
-<wire x1="30.48" y1="81.28" x2="30.48" y2="73.66" width="0.1524" layer="91" curve="180"/>
 <pinref part="IC2" gate="A" pin="OUT"/>
 <pinref part="R16" gate="G$1" pin="1"/>
 <junction x="154.94" y="134.62"/>
-<pinref part="U1" gate="U1" pin="(RX/MISO/ADC5)PA5"/>
-<wire x1="30.48" y1="73.66" x2="45.72" y2="73.66" width="0.1524" layer="91"/>
+<wire x1="154.94" y1="104.14" x2="35.56" y2="104.14" width="0.1524" layer="91"/>
+<wire x1="35.56" y1="104.14" x2="35.56" y2="78.74" width="0.1524" layer="91"/>
+<wire x1="35.56" y1="78.74" x2="48.26" y2="78.74" width="0.1524" layer="91"/>
 </segment>
 </net>
@@
 <segment>
 <wire x1="7.62" y1="88.9" x2="7.62" y2="83.82" width="0.1524" layer="91"/>
-<wire x1="45.72" y1="78.74" x2="22.86" y2="78.74" width="0.1524" layer="91"/>
-<wire x1="22.86" y1="78.74" x2="22.86" y2="83.82" width="0.1524" layer="91"/>
 <wire x1="22.86" y1="83.82" x2="7.62" y2="83.82" width="0.1524" layer="91"/>
 <wire x1="7.62" y1="88.9" x2="7.62" y2="86.36" width="0.1524" layer="91"/>
@@
 <pinref part="OK3" gate="A" pin="COL"/>
 <pinref part="R1" gate="G$1" pin="1"/>
-<pinref part="U1" gate="U1" pin="(ADC7)PA7"/>
+<wire x1="22.86" y1="83.82" x2="22.86" y2="76.2" width="0.1524" layer="91"/>
+<pinref part="U1" gate="U1" pin="(TX/SDA/MOSI/ADC6)PA6"/>
+<wire x1="22.86" y1="76.2" x2="45.72" y2="76.2" width="0.1524" layer="91"/>
 </segment>
 </net>
@@
 <pinref part="R14" gate="G$1" pin="1"/>
 <wire x1="25.4" y1="5.08" x2="25.4" y2="71.12" width="0.1524" layer="91"/>
-<wire x1="25.4" y1="71.12" x2="33.02" y2="71.12" width="0.1524" layer="91"/>
-<wire x1="33.02" y1="71.12" x2="35.56" y2="71.12" width="0.1524" layer="91"/>
-<wire x1="35.56" y1="71.12" x2="48.26" y2="71.12" width="0.1524" layer="91"/>
-</segment>
-</net>
-<net name="N$12" class="0">
-<segment>
-<wire x1="25.4" y1="35.56" x2="25.4" y2="5.08" width="0.1524" layer="91"/>
-</segment>
-<segment>
-<wire x1="25.4" y1="35.56" x2="25.4" y2="5.08" width="0.1524" layer="91"/>
+<wire x1="25.4" y1="71.12" x2="48.26" y2="71.12" width="0.1524" layer="91"/>
 </segment>
 </net>
@@
 <wire x1="104.14" y1="81.28" x2="88.9" y2="81.28" width="0.1524" layer="91"/>
 <wire x1="88.9" y1="81.28" x2="88.9" y2="53.34" width="0.1524" layer="91"/>
-<wire x1="88.9" y1="53.34" x2="33.02" y2="53.34" width="0.1524" layer="91"/>
-<wire x1="33.02" y1="53.34" x2="33.02" y2="63.5" width="0.1524" layer="91"/>
+<wire x1="88.9" y1="53.34" x2="43.18" y2="53.34" width="0.1524" layer="91"/>
+<wire x1="43.18" y1="53.34" x2="43.18" y2="63.5" width="0.1524" layer="91"/>
 <pinref part="U1" gate="U1" pin="(ADC1)PA1"/>
-<wire x1="33.02" y1="63.5" x2="45.72" y2="63.5" width="0.1524" layer="91"/>
-</segment>
-</net>
+<wire x1="43.18" y1="63.5" x2="45.72" y2="63.5" width="0.1524" layer="91"/>
+</segment>
+</net>

Commit message: schematic changes
Parts:
- added R8: 2k, resistor:R-EU_0613/5V
- R4, R7: value (none) -> 2k
Connections:
- net +12V: no longer R16.2
- net CPU-BOARD: now also IC2.OUT, R16.1; no longer IC2.+IN, SENS-1.P$1
- net ENTRY-BOARD: now also R16.2, R2.E, R8.2; no longer R4.2
- net N$1: now also R4.2
- net N$4: now also IC2.+IN, R8.1, SENS-1.P$1; no longer IC2.OUT, R16.1
- net PASSINGBEAM-ON: now also R4.1
Other:
- moved on the sheet: R4, R7
Changed lines of the file:
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@@
 <part name="R6" library="resistor" deviceset="R-EU_" device="0613/5V"/>
 <part name="SUPPLY17" library="supply2" deviceset="GND" device=""/>
-<part name="R4" library="resistor" deviceset="R-EU_" device="0613/5V"/>
-<part name="R7" library="resistor" deviceset="R-EU_" device="0613/5V"/>
 <part name="R10" library="resistor" deviceset="R-EU_" device="0613/5V" value="2k"/>
 <part name="R11" library="resistor" deviceset="R-EU_" device="0613/5V" value="2k"/>
@@
 <part name="DWIRE" library="con-lstb" deviceset="MA03-2" device=""/>
 <part name="SUPPLY25" library="supply2" deviceset="GND" device=""/>
+<part name="R4" library="resistor" deviceset="R-EU_" device="0613/5V" value="2k"/>
+<part name="R7" library="resistor" deviceset="R-EU_" device="0613/5V" value="2k"/>
+<part name="R8" library="resistor" deviceset="R-EU_" device="0613/5V" value="2k"/>
 </parts>
 <sheets>
@@
 <instance part="R6" gate="G$1" x="134.62" y="17.78"/>
 <instance part="SUPPLY17" gate="GND" x="111.76" y="78.74"/>
-<instance part="R4" gate="G$1" x="93.98" y="152.4" rot="R90"/>
-<instance part="R7" gate="G$1" x="88.9" y="152.4" rot="R90"/>
 <instance part="R10" gate="G$1" x="-15.24" y="86.36"/>
 <instance part="R11" gate="G$1" x="-15.24" y="48.26"/>
@@
 <instance part="R15" gate="G$1" x="-12.7" y="7.62"/>
 <instance part="R16" gate="G$1" x="154.94" y="139.7" rot="R90"/>
-<instance part="SUPPLY22" gate="+12V" x="154.94" y="147.32"/>
+<instance part="SUPPLY22" gate="+12V" x="154.94" y="154.94"/>
 <instance part="SUPPLY23" gate="+12V" x="132.08" y="63.5"/>
 <instance part="SUPPLY24" gate="GND" x="139.7" y="53.34"/>
 <instance part="DWIRE" gate="1" x="124.46" y="58.42" rot="R180"/>
 <instance part="SUPPLY25" gate="GND" x="-66.04" y="114.3"/>
+<instance part="R4" gate="G$1" x="-15.24" y="48.26"/>
+<instance part="R7" gate="G$1" x="132.08" y="157.48"/>
+<instance part="R8" gate="G$1" x="132.08" y="149.86"/>
 </instances>
 <busses>
@@
 <pinref part="R14" gate="G$1" pin="2"/>
 <pinref part="SUPPLY20" gate="+12V" pin="+12V"/>
-</segment>
-<segment>
-<pinref part="R16" gate="G$1" pin="2"/>
-<pinref part="SUPPLY22" gate="+12V" pin="+12V"/>
 </segment>
 <segment>
@@
 <wire x1="109.22" y1="116.84" x2="109.22" y2="127" width="0.1524" layer="91"/>
 <wire x1="109.22" y1="127" x2="116.84" y2="127" width="0.1524" layer="91"/>
+<pinref part="SENS-1" gate="G$1" pin="P$4"/>
+<wire x1="88.9" y1="127" x2="88.9" y2="116.84" width="0.1524" layer="91"/>
+<wire x1="109.22" y1="116.84" x2="88.9" y2="116.84" width="0.1524" layer="91"/>
 <wire x1="93.98" y1="129.54" x2="93.98" y2="127" width="0.1524" layer="91"/>
 <pinref part="SENS-1" gate="G$1" pin="P$2"/>
-<wire x1="93.98" y1="127" x2="93.98" y2="116.84" width="0.1524" layer="91"/>
-<wire x1="88.9" y1="116.84" x2="93.98" y2="116.84" width="0.1524" layer="91"/>
-<pinref part="SENS-1" gate="G$1" pin="P$4"/>
-<wire x1="88.9" y1="127" x2="88.9" y2="116.84" width="0.1524" layer="91"/>
-<wire x1="109.22" y1="116.84" x2="93.98" y2="116.84" width="0.1524" layer="91"/>
+<wire x1="88.9" y1="127" x2="93.98" y2="127" width="0.1524" layer="91"/>
 </segment>
 <segment>
@@
 </segment>
 </net>
-<net name="N$4" class="0">
+<net name="CPU-BOARD" class="0">
 <segment>
 <wire x1="154.94" y1="134.62" x2="154.94" y2="104.14" width="0.1524" layer="91"/>
@@
 <wire x1="35.56" y1="104.14" x2="35.56" y2="78.74" width="0.1524" layer="91"/>
 <wire x1="35.56" y1="78.74" x2="48.26" y2="78.74" width="0.1524" layer="91"/>
+<label x="139.7" y="165.1" size="3.048" layer="95"/>
 </segment>
 </net>
@@
 <pinref part="OK4" gate="A" pin="A"/>
 <pinref part="R11" gate="G$1" pin="2"/>
+<pinref part="R4" gate="G$1" pin="2"/>
+<junction x="-10.16" y="48.26"/>
+<pinref part="R4" gate="G$1" pin="2"/>
 </segment>
 </net>
@@
 <pinref part="S2" gate="1" pin="P"/>
 <wire x1="-20.32" y1="48.26" x2="-55.88" y2="48.26" width="0.1524" layer="91"/>
+<pinref part="R4" gate="G$1" pin="1"/>
+<junction x="-20.32" y="48.26"/>
 </segment>
 <segment>
@@
 <pinref part="SUPPLY1" gate="+12V" pin="+12V"/>
 <pinref part="C1" gate="G$1" pin="+"/>
-</segment>
-</net>
-<net name="N$2" class="0">
-<segment>
-<pinref part="R7" gate="G$1" pin="1"/>
-<pinref part="SENS-1" gate="G$1" pin="P$3"/>
 </segment>
 </net>
@@
 <pinref part="U1" gate="U1" pin="(ADC1)PA1"/>
 <wire x1="43.18" y1="63.5" x2="45.72" y2="63.5" width="0.1524" layer="91"/>
-</segment>
-</net>
-<net name="CPU-BOARD" class="0">
-<segment>
-<wire x1="114.3" y1="147.32" x2="119.38" y2="147.32" width="0.1524" layer="91" curve="-180"/>
-<wire x1="124.46" y1="147.32" x2="124.46" y2="137.16" width="0.1524" layer="91"/>
-<pinref part="IC2" gate="A" pin="+IN"/>
-<wire x1="119.38" y1="147.32" x2="124.46" y2="147.32" width="0.1524" layer="91"/>
-<pinref part="SENS-1" gate="G$1" pin="P$1"/>
-<wire x1="114.3" y1="147.32" x2="93.98" y2="147.32" width="0.1524" layer="91"/>
-<label x="111.76" y="165.1" size="3.048" layer="95"/>
 </segment>
 </net>
@@
 <wire x1="7.62" y1="124.46" x2="10.16" y2="124.46" width="0.1524" layer="91"/>
 <pinref part="IC1" gate="A1" pin="VO"/>
-<pinref part="R4" gate="G$1" pin="2"/>
-<wire x1="35.56" y1="157.48" x2="88.9" y2="157.48" width="0.1524" layer="91"/>
-<wire x1="93.98" y1="157.48" x2="88.9" y2="157.48" width="0.1524" layer="91"/>
-<pinref part="R7" gate="G$1" pin="2"/>
-<wire x1="93.98" y1="157.48" x2="116.84" y2="157.48" width="0.1524" layer="91"/>
-<wire x1="116.84" y1="157.48" x2="116.84" y2="134.62" width="0.1524" layer="91"/>
-<wire x1="35.56" y1="157.48" x2="35.56" y2="124.46" width="0.1524" layer="91"/>
+<wire x1="35.56" y1="167.64" x2="35.56" y2="124.46" width="0.1524" layer="91"/>
 <wire x1="35.56" y1="124.46" x2="22.86" y2="124.46" width="0.1524" layer="91"/>
 <label x="7.62" y="157.48" size="3.302" layer="95" rot="MR0"/>
-</segment>
-</net>
+<wire x1="35.56" y1="167.64" x2="137.16" y2="167.64" width="0.1524" layer="91"/>
+<wire x1="137.16" y1="167.64" x2="137.16" y2="157.48" width="0.1524" layer="91"/>
+<pinref part="R16" gate="G$1" pin="2"/>
+<pinref part="SUPPLY22" gate="+12V" pin="+12V"/>
+<wire x1="137.16" y1="157.48" x2="137.16" y2="149.86" width="0.1524" layer="91"/>
+<wire x1="137.16" y1="149.86" x2="137.16" y2="144.78" width="0.1524" layer="91"/>
+<wire x1="154.94" y1="152.4" x2="154.94" y2="144.78" width="0.1524" layer="91"/>
+<wire x1="137.16" y1="144.78" x2="154.94" y2="144.78" width="0.1524" layer="91"/>
+<wire x1="137.16" y1="144.78" x2="116.84" y2="144.78" width="0.1524" layer="91"/>
+<pinref part="R2" gate="1" pin="E"/>
+<wire x1="116.84" y1="144.78" x2="116.84" y2="137.16" width="0.1524" layer="91"/>
+<pinref part="R7" gate="G$1" pin="2"/>
+<junction x="137.16" y="157.48"/>
+<pinref part="R8" gate="G$1" pin="2"/>
+<junction x="137.16" y="149.86"/>
+</segment>
+</net>
+<net name="N$2" class="0">
+<segment>
+<pinref part="R7" gate="G$1" pin="1"/>
+<wire x1="127" y1="157.48" x2="88.9" y2="157.48" width="0.1524" layer="91"/>
+<pinref part="SENS-1" gate="G$1" pin="P$3"/>
+<wire x1="88.9" y1="157.48" x2="88.9" y2="147.32" width="0.1524" layer="91"/>
+</segment>
+</net>
+<net name="N$4" class="0">
+<segment>
+<pinref part="R8" gate="G$1" pin="1"/>
+<wire x1="127" y1="149.86" x2="109.22" y2="149.86" width="0.1524" layer="91"/>
+<pinref part="SENS-1" gate="G$1" pin="P$1"/>
+<wire x1="109.22" y1="149.86" x2="93.98" y2="149.86" width="0.1524" layer="91"/>
+<wire x1="93.98" y1="149.86" x2="93.98" y2="147.32" width="0.1524" layer="91"/>
+<wire x1="109.22" y1="149.86" x2="109.22" y2="137.16" width="0.1524" layer="91"/>
+<wire x1="109.22" y1="137.16" x2="114.3" y2="137.16" width="0.1524" layer="91"/>
+<pinref part="IC2" gate="A" pin="+IN"/>
+<wire x1="124.46" y1="137.16" x2="119.38" y2="137.16" width="0.1524" layer="91"/>
+<wire x1="114.3" y1="137.16" x2="119.38" y2="137.16" width="0.1524" layer="91" curve="-180"/>
+</segment>
+</net>

Commit message: schematic changes
Connections:
- net CPU-BOARD: now also U1.(INT0)PB2
- net LED-BOARD: now also U1.(ADC1)PA1
- net N$10: no longer U1.(ADC3)PA3
- net N$15: now also U1.(XTAL2)PB1; no longer U1.(TX/SDA/MOSI/ADC6)PA6
- net N$19: now also U1.(ADC0)PA0; no longer U1.(ADC1)PA1
- net N$5: now also U1.(ADC3)PA3
- net N$6: now also U1.(XTAL1)PB0; no longer U1.(RX/MISO/ADC5)PA5
Changed lines of the file:
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@@
 <pinref part="OK4" gate="A" pin="COL"/>
 <pinref part="R3" gate="G$1" pin="1"/>
-<wire x1="22.86" y1="45.72" x2="22.86" y2="73.66" width="0.1524" layer="91"/>
-<pinref part="U1" gate="U1" pin="(RX/MISO/ADC5)PA5"/>
-<wire x1="45.72" y1="73.66" x2="38.1" y2="73.66" width="0.1524" layer="91"/>
-<wire x1="38.1" y1="73.66" x2="35.56" y2="73.66" width="0.1524" layer="91"/>
-<wire x1="22.86" y1="73.66" x2="35.56" y2="73.66" width="0.1524" layer="91"/>
+<wire x1="22.86" y1="45.72" x2="22.86" y2="81.28" width="0.1524" layer="91"/>
+<wire x1="22.86" y1="81.28" x2="35.56" y2="81.28" width="0.1524" layer="91"/>
+<wire x1="35.56" y1="81.28" x2="35.56" y2="83.82" width="0.1524" layer="91"/>
+<pinref part="U1" gate="U1" pin="(XTAL1)PB0"/>
+<wire x1="35.56" y1="83.82" x2="45.72" y2="83.82" width="0.1524" layer="91"/>
 </segment>
 </net>
@@
 <net name="N$10" class="0">
 <segment>
-<wire x1="38.1" y1="68.58" x2="38.1" y2="17.78" width="0.1524" layer="91"/>
-<wire x1="38.1" y1="17.78" x2="129.54" y2="17.78" width="0.1524" layer="91"/>
+<wire x1="35.56" y1="17.78" x2="129.54" y2="17.78" width="0.1524" layer="91"/>
 <pinref part="R6" gate="G$1" pin="1"/>
-<pinref part="U1" gate="U1" pin="(ADC3)PA3"/>
-<wire x1="38.1" y1="68.58" x2="45.72" y2="68.58" width="0.1524" layer="91"/>
+<wire x1="35.56" y1="17.78" x2="35.56" y2="66.04" width="0.1524" layer="91"/>
+<wire x1="35.56" y1="66.04" x2="48.26" y2="66.04" width="0.1524" layer="91"/>
 </segment>
 </net>
 <net name="LED-BOARD" class="0">
 <segment>
-<wire x1="40.64" y1="66.04" x2="40.64" y2="27.94" width="0.1524" layer="91"/>
 <wire x1="40.64" y1="27.94" x2="129.54" y2="27.94" width="0.1524" layer="91"/>
 <pinref part="R5" gate="G$1" pin="1"/>
-<wire x1="40.64" y1="66.04" x2="48.26" y2="66.04" width="0.1524" layer="91"/>
 <label x="129.54" y="38.1" size="3.048" layer="95"/>
+<wire x1="40.64" y1="27.94" x2="40.64" y2="63.5" width="0.1524" layer="91"/>
+<pinref part="U1" gate="U1" pin="(ADC1)PA1"/>
+<wire x1="40.64" y1="63.5" x2="45.72" y2="63.5" width="0.1524" layer="91"/>
 </segment>
 </net>
@@
 <junction x="154.94" y="134.62"/>
 <wire x1="154.94" y1="104.14" x2="35.56" y2="104.14" width="0.1524" layer="91"/>
-<wire x1="35.56" y1="104.14" x2="35.56" y2="78.74" width="0.1524" layer="91"/>
-<wire x1="35.56" y1="78.74" x2="48.26" y2="78.74" width="0.1524" layer="91"/>
 <label x="139.7" y="165.1" size="3.048" layer="95"/>
+<wire x1="35.56" y1="104.14" x2="35.56" y2="88.9" width="0.1524" layer="91"/>
+<pinref part="U1" gate="U1" pin="(INT0)PB2"/>
+<wire x1="35.56" y1="88.9" x2="45.72" y2="88.9" width="0.1524" layer="91"/>
 </segment>
 </net>
@@
 <segment>
 <wire x1="7.62" y1="88.9" x2="7.62" y2="83.82" width="0.1524" layer="91"/>
-<wire x1="22.86" y1="83.82" x2="7.62" y2="83.82" width="0.1524" layer="91"/>
 <wire x1="7.62" y1="88.9" x2="7.62" y2="86.36" width="0.1524" layer="91"/>
 <junction x="7.62" y="88.9"/>
 <pinref part="OK3" gate="A" pin="COL"/>
 <pinref part="R1" gate="G$1" pin="1"/>
-<wire x1="22.86" y1="83.82" x2="22.86" y2="76.2" width="0.1524" layer="91"/>
-<pinref part="U1" gate="U1" pin="(TX/SDA/MOSI/ADC6)PA6"/>
-<wire x1="22.86" y1="76.2" x2="45.72" y2="76.2" width="0.1524" layer="91"/>
+<wire x1="7.62" y1="83.82" x2="33.02" y2="83.82" width="0.1524" layer="91"/>
+<wire x1="33.02" y1="83.82" x2="33.02" y2="86.36" width="0.1524" layer="91"/>
+<pinref part="U1" gate="U1" pin="(XTAL2)PB1"/>
+<wire x1="33.02" y1="86.36" x2="45.72" y2="86.36" width="0.1524" layer="91"/>
 </segment>
 </net>
@@
 <pinref part="OK1" gate="A" pin="COL"/>
 <pinref part="R14" gate="G$1" pin="1"/>
-<wire x1="25.4" y1="5.08" x2="25.4" y2="71.12" width="0.1524" layer="91"/>
-<wire x1="25.4" y1="71.12" x2="48.26" y2="71.12" width="0.1524" layer="91"/>
+<wire x1="25.4" y1="5.08" x2="25.4" y2="68.58" width="0.1524" layer="91"/>
+<pinref part="U1" gate="U1" pin="(ADC3)PA3"/>
+<wire x1="25.4" y1="68.58" x2="45.72" y2="68.58" width="0.1524" layer="91"/>
 </segment>
 </net>
@@
 <wire x1="88.9" y1="81.28" x2="88.9" y2="53.34" width="0.1524" layer="91"/>
 <wire x1="88.9" y1="53.34" x2="43.18" y2="53.34" width="0.1524" layer="91"/>
-<wire x1="43.18" y1="53.34" x2="43.18" y2="63.5" width="0.1524" layer="91"/>
-<pinref part="U1" gate="U1" pin="(ADC1)PA1"/>
-<wire x1="43.18" y1="63.5" x2="45.72" y2="63.5" width="0.1524" layer="91"/>
+<wire x1="43.18" y1="53.34" x2="43.18" y2="60.96" width="0.1524" layer="91"/>
+<pinref part="U1" gate="U1" pin="(ADC0)PA0"/>
+<wire x1="43.18" y1="60.96" x2="45.72" y2="60.96" width="0.1524" layer="91"/>
 </segment>
 </net>
