File: KsbSchematics/KsbSchematics/KsbLightSensorSchematic.sch (EAGLE design)
At the start: 30 parts, among them IC1 7805L, IC2 LM311N, U1 ATTINY84

Commit message: schematic changes
Connections:
- removed net N$10: R6.1
- removed net N$19: SG1.1, U1.(ADC0)PA0
- new net N$12: R6.1, U1.(ADC1)PA1
- new net N$14: SG1.1
- net GND: now also IC2.GND
- net LED-BOARD: now also U1.(ADC0)PA0; no longer U1.(ADC1)PA1
Changed lines of the file:
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@@
 <part name="R7" library="resistor" deviceset="R-EU_" device="0613/5V" value="2k"/>
 <part name="R8" library="resistor" deviceset="R-EU_" device="0613/5V" value="2k"/>
+<part name="SUPPLY26" library="supply2" deviceset="GND" device=""/>
 </parts>
 <sheets>
@@
 <instance part="R7" gate="G$1" x="132.08" y="157.48"/>
 <instance part="R8" gate="G$1" x="132.08" y="149.86"/>
+<instance part="SUPPLY26" gate="GND" x="132.08" y="124.46"/>
 </instances>
 <busses>
@@
 <pinref part="SUPPLY17" gate="GND" pin="GND"/>
 </segment>
+<segment>
+<pinref part="IC2" gate="A" pin="GND"/>
+<pinref part="SUPPLY26" gate="GND" pin="GND"/>
+</segment>
 </net>
 <net name="N$6" class="0">
@@
 </segment>
 </net>
-<net name="N$10" class="0">
-<segment>
-<wire x1="35.56" y1="17.78" x2="129.54" y2="17.78" width="0.1524" layer="91"/>
-<pinref part="R6" gate="G$1" pin="1"/>
-<wire x1="35.56" y1="17.78" x2="35.56" y2="66.04" width="0.1524" layer="91"/>
-<wire x1="35.56" y1="66.04" x2="48.26" y2="66.04" width="0.1524" layer="91"/>
-</segment>
-</net>
 <net name="LED-BOARD" class="0">
 <segment>
@@
 <pinref part="R5" gate="G$1" pin="1"/>
 <label x="129.54" y="38.1" size="3.048" layer="95"/>
-<wire x1="40.64" y1="27.94" x2="40.64" y2="63.5" width="0.1524" layer="91"/>
-<pinref part="U1" gate="U1" pin="(ADC1)PA1"/>
-<wire x1="40.64" y1="63.5" x2="45.72" y2="63.5" width="0.1524" layer="91"/>
+<wire x1="40.64" y1="27.94" x2="40.64" y2="60.96" width="0.1524" layer="91"/>
+<pinref part="U1" gate="U1" pin="(ADC0)PA0"/>
+<wire x1="43.18" y1="60.96" x2="45.72" y2="60.96" width="0.1524" layer="91"/>
+<wire x1="40.64" y1="60.96" x2="45.72" y2="60.96" width="0.1524" layer="91"/>
 </segment>
 </net>
@@
 <pinref part="S2" gate="1" pin="O"/>
 <label x="-76.2" y="50.8" size="2.54" layer="95" rot="R180"/>
-</segment>
-</net>
-<net name="N$19" class="0">
-<segment>
-<pinref part="SG1" gate="G$1" pin="1"/>
-<wire x1="104.14" y1="81.28" x2="88.9" y2="81.28" width="0.1524" layer="91"/>
-<wire x1="88.9" y1="81.28" x2="88.9" y2="53.34" width="0.1524" layer="91"/>
-<wire x1="88.9" y1="53.34" x2="43.18" y2="53.34" width="0.1524" layer="91"/>
-<wire x1="43.18" y1="53.34" x2="43.18" y2="60.96" width="0.1524" layer="91"/>
-<pinref part="U1" gate="U1" pin="(ADC0)PA0"/>
-<wire x1="43.18" y1="60.96" x2="45.72" y2="60.96" width="0.1524" layer="91"/>
 </segment>
 </net>
@@
 </segment>
 </net>
+<net name="N$12" class="0">
+<segment>
+<pinref part="U1" gate="U1" pin="(ADC1)PA1"/>
+<wire x1="38.1" y1="63.5" x2="40.64" y2="63.5" width="0.1524" layer="91"/>
+<pinref part="R6" gate="G$1" pin="1"/>
+<wire x1="43.18" y1="63.5" x2="45.72" y2="63.5" width="0.1524" layer="91"/>
+<wire x1="129.54" y1="17.78" x2="38.1" y2="17.78" width="0.1524" layer="91"/>
+<wire x1="38.1" y1="17.78" x2="38.1" y2="63.5" width="0.1524" layer="91"/>
+<wire x1="40.64" y1="63.5" x2="43.18" y2="63.5" width="0.1524" layer="91"/>
+</segment>
+</net>
+<net name="N$14" class="0">
+<segment>
+<wire x1="35.56" y1="66.04" x2="48.26" y2="66.04" width="0.1524" layer="91"/>
+<pinref part="SG1" gate="G$1" pin="1"/>
+<wire x1="104.14" y1="81.28" x2="88.9" y2="81.28" width="0.1524" layer="91"/>
+<wire x1="88.9" y1="81.28" x2="88.9" y2="53.34" width="0.1524" layer="91"/>
+<wire x1="88.9" y1="53.34" x2="43.18" y2="53.34" width="0.1524" layer="91"/>
+<wire x1="43.18" y1="53.34" x2="35.56" y2="53.34" width="0.1524" layer="91" curve="-180"/>
+<wire x1="35.56" y1="66.04" x2="35.56" y2="53.34" width="0.1524" layer="91"/>
+</segment>
+</net>

Commit message: schematic changes
Parts:
- added U2: ATTINY84, SparkFun-IC-Microcontroller:ATTINY84
Connections:
- new net N$11: U1.VCC, U2.VCC
- new net N$17: U1.(SCL/SCK/ADC4)PA4, U2.(SCL/SCK/ADC4)PA4
- new net N$18: U1.(RX/MISO/ADC5)PA5, U2.(RX/MISO/ADC5)PA5
- new net N$20: U1.(TX/SDA/MOSI/ADC6)PA6, U2.(TX/SDA/MOSI/ADC6)PA6
- new net N$21: U1.(ADC7)PA7, U2.(ADC7)PA7
- new net N$22: U1.GND, U2.GND
- net CPU-BOARD: now also U2.(INT0)PB2
- net LED-BOARD: now also U2.(ADC0)PA0
- net N$12: now also U2.(ADC1)PA1
- net N$14: now also U2.(ADC2)PA2
- net N$15: now also U2.(XTAL2)PB1
- net N$5: now also U2.(ADC3)PA3
- net N$6: now also U2.(XTAL1)PB0
- net N$7: now also U2.(!RESET!)PB3
Changed lines of the file:
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@@
 <part name="R8" library="resistor" deviceset="R-EU_" device="0613/5V" value="2k"/>
 <part name="SUPPLY26" library="supply2" deviceset="GND" device=""/>
+<part name="U2" library="SparkFun-IC-Microcontroller" deviceset="ATTINY84" device="" value="ATTINY84"/>
 </parts>
 <sheets>
@@
 <instance part="R8" gate="G$1" x="132.08" y="149.86"/>
 <instance part="SUPPLY26" gate="GND" x="132.08" y="124.46"/>
+<instance part="U2" gate="U1" x="63.5" y="76.2" rot="MR0"/>
 </instances>
 <busses>
@@
 <pinref part="R2" gate="1" pin="A"/>
 <pinref part="SUPPLY6" gate="GND" pin="GND"/>
-<wire x1="109.22" y1="116.84" x2="109.22" y2="127" width="0.1524" layer="91"/>
+<wire x1="109.22" y1="116.84" x2="109.22" y2="119.38" width="0.1524" layer="91"/>
+<wire x1="109.22" y1="119.38" x2="109.22" y2="127" width="0.1524" layer="91"/>
 <wire x1="109.22" y1="127" x2="116.84" y2="127" width="0.1524" layer="91"/>
 <pinref part="SENS-1" gate="G$1" pin="P$4"/>
@@
 <wire x1="93.98" y1="129.54" x2="93.98" y2="127" width="0.1524" layer="91"/>
 <pinref part="SENS-1" gate="G$1" pin="P$2"/>
-<wire x1="88.9" y1="127" x2="93.98" y2="127" width="0.1524" layer="91"/>
+<wire x1="93.98" y1="127" x2="93.98" y2="119.38" width="0.1524" layer="91"/>
+<wire x1="93.98" y1="119.38" x2="109.22" y2="119.38" width="0.1524" layer="91"/>
 </segment>
 <segment>
@@
 <pinref part="U1" gate="U1" pin="(XTAL1)PB0"/>
 <wire x1="35.56" y1="83.82" x2="45.72" y2="83.82" width="0.1524" layer="91"/>
+<pinref part="U2" gate="U1" pin="(XTAL1)PB0"/>
+<junction x="45.72" y="83.82"/>
 </segment>
 </net>
@@
 <wire x1="43.18" y1="60.96" x2="45.72" y2="60.96" width="0.1524" layer="91"/>
 <wire x1="40.64" y1="60.96" x2="45.72" y2="60.96" width="0.1524" layer="91"/>
+<pinref part="U2" gate="U1" pin="(ADC0)PA0"/>
+<junction x="45.72" y="60.96"/>
 </segment>
 </net>
@@
 <pinref part="U1" gate="U1" pin="(INT0)PB2"/>
 <wire x1="35.56" y1="88.9" x2="45.72" y2="88.9" width="0.1524" layer="91"/>
+<pinref part="U2" gate="U1" pin="(INT0)PB2"/>
+<junction x="45.72" y="88.9"/>
 </segment>
 </net>
@@
 <pinref part="U1" gate="U1" pin="(XTAL2)PB1"/>
 <wire x1="33.02" y1="86.36" x2="45.72" y2="86.36" width="0.1524" layer="91"/>
+<pinref part="U2" gate="U1" pin="(XTAL2)PB1"/>
+<junction x="45.72" y="86.36"/>
 </segment>
 </net>
@@
 <pinref part="U1" gate="U1" pin="(ADC3)PA3"/>
 <wire x1="25.4" y1="68.58" x2="45.72" y2="68.58" width="0.1524" layer="91"/>
+<pinref part="U2" gate="U1" pin="(ADC3)PA3"/>
+<junction x="45.72" y="68.58"/>
 </segment>
 </net>
@@
 <wire x1="109.22" y1="55.88" x2="116.84" y2="55.88" width="0.1524" layer="91"/>
 <wire x1="109.22" y1="71.12" x2="109.22" y2="55.88" width="0.1524" layer="91"/>
+<pinref part="U2" gate="U1" pin="(!RESET!)PB3"/>
+<junction x="45.72" y="91.44"/>
 </segment>
 </net>
@@
 <wire x1="38.1" y1="17.78" x2="38.1" y2="63.5" width="0.1524" layer="91"/>
 <wire x1="40.64" y1="63.5" x2="43.18" y2="63.5" width="0.1524" layer="91"/>
+<pinref part="U2" gate="U1" pin="(ADC1)PA1"/>
+<junction x="45.72" y="63.5"/>
 </segment>
 </net>
 <net name="N$14" class="0">
 <segment>
-<wire x1="35.56" y1="66.04" x2="48.26" y2="66.04" width="0.1524" layer="91"/>
+<wire x1="35.56" y1="66.04" x2="45.72" y2="66.04" width="0.1524" layer="91"/>
 <pinref part="SG1" gate="G$1" pin="1"/>
+<wire x1="45.72" y1="66.04" x2="48.26" y2="66.04" width="0.1524" layer="91"/>
 <wire x1="104.14" y1="81.28" x2="88.9" y2="81.28" width="0.1524" layer="91"/>
 <wire x1="88.9" y1="81.28" x2="88.9" y2="53.34" width="0.1524" layer="91"/>
@@
 <wire x1="43.18" y1="53.34" x2="35.56" y2="53.34" width="0.1524" layer="91" curve="-180"/>
 <wire x1="35.56" y1="66.04" x2="35.56" y2="53.34" width="0.1524" layer="91"/>
-</segment>
-</net>
+<pinref part="U2" gate="U1" pin="(ADC2)PA2"/>
+<junction x="45.72" y="66.04"/>
+</segment>
+</net>
+<net name="N$11" class="0">
+<segment>
+<pinref part="U1" gate="U1" pin="VCC"/>
+<pinref part="U2" gate="U1" pin="VCC"/>
+</segment>
+</net>
+<net name="N$17" class="0">
+<segment>
+<pinref part="U1" gate="U1" pin="(SCL/SCK/ADC4)PA4"/>
+<pinref part="U2" gate="U1" pin="(SCL/SCK/ADC4)PA4"/>
+</segment>
+</net>
+<net name="N$18" class="0">
+<segment>
+<pinref part="U1" gate="U1" pin="(RX/MISO/ADC5)PA5"/>
+<pinref part="U2" gate="U1" pin="(RX/MISO/ADC5)PA5"/>
+</segment>
+</net>
+<net name="N$20" class="0">
+<segment>
+<pinref part="U1" gate="U1" pin="(TX/SDA/MOSI/ADC6)PA6"/>
+<pinref part="U2" gate="U1" pin="(TX/SDA/MOSI/ADC6)PA6"/>
+</segment>
+</net>
+<net name="N$21" class="0">
+<segment>
+<pinref part="U1" gate="U1" pin="(ADC7)PA7"/>
+<pinref part="U2" gate="U1" pin="(ADC7)PA7"/>
+</segment>
+</net>
+<net name="N$22" class="0">
+<segment>
+<pinref part="U1" gate="U1" pin="GND"/>
+<pinref part="U2" gate="U1" pin="GND"/>
+</segment>
+</net>
