File: KsbSchematics/KsbSchematics/KsbLightSensorSchematic.sch (EAGLE design)
At the start: 31 parts, among them IC1 7805L, IC2 LM311N, U1 ATTINY84, U2 ATTINY84

Commit message: tested so far ok
Parts:
- added S4: (no value), switch-omron:31-XX
Connections:
- net GND: now also S4.S
- net N$21: now also S4.P
Changed lines of the file:
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@@
 <part name="SUPPLY26" library="supply2" deviceset="GND" device=""/>
 <part name="U2" library="SparkFun-IC-Microcontroller" deviceset="ATTINY84" device="" value="ATTINY84"/>
+<part name="S4" library="switch-omron" deviceset="31-XX" device=""/>
+<part name="SUPPLY27" library="supply2" deviceset="GND" device=""/>
+<part name="SUPPLY28" library="supply2" deviceset="GND" device=""/>
 </parts>
 <sheets>
@@
 <plain>
 <rectangle x1="-40.64" y1="-5.08" x2="-38.1" y2="160.02" layer="91"/>
-<rectangle x1="-30.48" y1="-5.08" x2="27.94" y2="154.94" layer="207"/>
+<rectangle x1="-30.48" y1="-5.08" x2="27.94" y2="154.94" layer="207" rot="R180"/>
 <polygon width="0.1524" layer="207">
 <vertex x="104.14" y="109.22"/>
@@
 <instance part="SUPPLY26" gate="GND" x="132.08" y="124.46"/>
 <instance part="U2" gate="U1" x="63.5" y="76.2" rot="MR0"/>
+<instance part="S4" gate="1" x="48.26" y="0" rot="R270"/>
+<instance part="SUPPLY27" gate="GND" x="-66.04" y="43.18"/>
+<instance part="SUPPLY28" gate="GND" x="53.34" y="-2.54"/>
 </instances>
 <busses>
@@
 <pinref part="S2" gate="1" pin="S"/>
 <pinref part="SUPPLY11" gate="GND" pin="GND"/>
+<pinref part="SUPPLY27" gate="GND" pin="GND"/>
+<junction x="-66.04" y="45.72"/>
+<pinref part="SUPPLY27" gate="GND" pin="GND"/>
 </segment>
 <segment>
@@
 <pinref part="IC2" gate="A" pin="GND"/>
 <pinref part="SUPPLY26" gate="GND" pin="GND"/>
+</segment>
+<segment>
+<pinref part="S4" gate="1" pin="S"/>
+<pinref part="SUPPLY28" gate="GND" pin="GND"/>
 </segment>
 </net>
@@
 <pinref part="U1" gate="U1" pin="(ADC7)PA7"/>
 <pinref part="U2" gate="U1" pin="(ADC7)PA7"/>
-</segment>
-</net>
+<wire x1="45.72" y1="78.74" x2="33.02" y2="78.74" width="0.1524" layer="91"/>
+<wire x1="33.02" y1="78.74" x2="33.02" y2="71.12" width="0.1524" layer="91"/>
+<wire x1="33.02" y1="71.12" x2="33.02" y2="66.04" width="0.1524" layer="91" curve="180"/>
+<wire x1="33.02" y1="66.04" x2="33.02" y2="0" width="0.1524" layer="91"/>
+<pinref part="S4" gate="1" pin="P"/>
+<wire x1="33.02" y1="0" x2="43.18" y2="0" width="0.1524" layer="91"/>
+</segment>
+</net>
